File: pcb/pcb.brd (EAGLE design)
At the start: 160 x 100 mm, 7 parts, among them J1 22-27-2031-03, U1 RASPBERRY_PICOSMD-TH

Commit message: [PCB] Finished design subject to testing
Parts:
- removed C1: 1mF, SparkFun-Capacitors:CPOL-RADIAL-5MM-10MM
- removed J1: 22-27-2031-03, con-molex:6410-03
- added H1, H2, H3, H4: MOUNT-HOLE3.0, holes:3,0
- added L5V, LD, LG: LSP10, solpad:LSP10
- added R1, R2, R3, R4, R5: (no value), rcl:0207/7
- added S2, S3, S4: MOMENTARY-SWITCH-SPST-PTH-12MM, SparkFun-Switches:TACTILE_SWITCH_PTH_12MM
- U1: value RASPBERRY_PICOSMD-TH -> RASPBERRY_PICOTH; device RpiPico:PICO-PKG -> RpiPico:PICO-PKG-TH
- moved A2 111.9 mm to (58.4, 31.8), turned to 90 degrees
- moved S1 97.7 mm to (34.3, 30.5), flipped to the bottom, turned to 90 degrees
- moved D1 69.1 mm to (12.7, 30.5), turned to 90 degrees
- moved U1 62.3 mm to (34.3, 11.4), turned to 90 degrees
- moved A1 62.0 mm to (20.3, 31.8), turned to 270 degrees
Connections:
- removed net 3V3(OUT): U1.36, U1.P$36
- removed net 5V: A2.1, C1.+, D1.C, S1.2
- removed net N$1: A1.1, S1.3
- removed net VSYS: U1.39, U1.P$39
- new net 3V3: A2.1, R4.1, R5.1, S1.1, S2.1, S3.1, S4.1, U1.36
- new net LEDDATA: LD.MP, U1.1
- new net SW1: S1.2, U1.31
- new net SW4: R1.1, R2.1, R3.1, S2.3, S3.3, S4.3, U1.17, U1.19, U1.20
- new net VCC: A1.1, D1.C, L5V.MP, U1.39
- net GND: now also LG.MP, R1.2, R2.2, R3.2, S1.3; no longer C1.-, U1.P$13, U1.P$18, U1.P$23, U1.P$28, U1.P$3, U1.P$33, U1.P$38, U1.P$8
- net INT: now also U1.29
- net SCL: now also R5.2, U1.22
- net SDA: now also R4.2, U1.21
- net SWGND: no longer U1.P$42
- net VBUS: no longer U1.P$40
Routing:
- net 3V3: track 0.00 -> 123.5 mm
- net SW4: track 0.00 -> 72.4 mm
- net LEDDATA: track 0.00 -> 58.8 mm
- net INT: track 0.00 -> 34.9 mm
- net VCC: track 0.00 -> 32.6 mm
- net SCL: track 0.00 -> 23.3 mm
- net SDA: track 0.00 -> 16.1 mm
- net SW1: track 0.00 -> 10.7 mm
- added copper zone on layer 1, net GND
- added copper zone on layer 16, net GND
Other:
- board size 160 x 100 mm -> 88.9 x 40.6 mm
- board text added: "BRIGHT NESS"
- board text added: "JAROD <3 SEOHYUN 4 YEARS 2022"
- board text added: "MODE"
- board text added: "ON"
- board text added: "TIME"

Commit message: [PCB] Sent off for manufacturing
Parts:
- removed H1, H2, H3, H4: MOUNT-HOLE3.0, holes:3,0
Connections:
- new net SW2: R1.1, S2.3, U1.20
- new net SW3: R2.1, S3.3, U1.19
- net LEDDATA: now also U1.34; no longer U1.1
- net SCL: now also U1.27; no longer U1.22
- net SDA: now also U1.26; no longer U1.21
- net SW4: no longer R1.1, R2.1, S2.3, S3.3, U1.19, U1.20
Routing:
- net LEDDATA: track 58.8 -> 23.7 mm
- net SW4: track 72.4 -> 38.6 mm
- net 3V3: track 123.5 -> 90.0 mm
- net SW3: track 0.00 -> 24.0 mm
- net SW2: track 0.00 -> 8.26 mm
- net SCL: track 23.3 -> 25.1 mm
- net SDA: track 16.1 -> 17.1 mm
Other:
- board text added: "JAROD SEOHYUN 4 YEARS 2022"
- board text added: "OFF"
- board text removed: "JAROD <3 SEOHYUN 4 YEARS 2022"
