File: pcb/pcb.sch (EAGLE design)
At the start: 7 parts, among them J1 22-27-2031-03, U1 RASPBERRY_PICOSMD-TH

Commit message: [PCB] Finished design subject to testing
Parts:
- removed C1: 1mF, SparkFun-Capacitors:1000UF-RADIAL-5MM-25V-20%
- removed J1: 22-27-2031-03, con-molex:22-27-2031-03
- added H1, H2, H3, H4: MOUNT-HOLE3.0, holes:MOUNT-HOLE3.0
- added L5V, LD, LG: LSP10, solpad:LSP10
- added R1, R2, R3, R4, R5: (no value), rcl:R-EU_0207/7
- added S2, S3, S4: MOMENTARY-SWITCH-SPST-PTH-12MM, SparkFun-Switches:MOMENTARY-SWITCH-SPST-PTH-12MM
- U1: value RASPBERRY_PICOSMD-TH -> RASPBERRY_PICOTH; device RpiPico:RASPBERRY_PICOSMD-TH -> RpiPico:RASPBERRY_PICOTH
Connections:
- removed net 5V: A2.1, C1.+, D1.C, S1.P
- removed net N$1: A1.1, S1.S
- new net 3V3: A2.1, R4.1, R5.1, S1.O, S2.1, S3.1, S4.1, U1.3V3(OUT)
- new net LEDDATA: LD.MP, U1.GP0
- new net SW1: S1.P, U1.GP26
- new net SW4: R1.1, R2.1, R3.1, S2.2, S3.2, S4.2, U1.GP13, U1.GP14, U1.GP15
- new net VCC: A1.1, D1.C, L5V.MP, U1.VSYS
- net GND: now also LG.MP, R1.2, R2.2, R3.2, S1.S, U1.GND; no longer C1.-
- net INT: now also U1.GP22
- net SCL: now also R5.2, U1.GP17
- net SDA: now also R4.2, U1.GP16
Other:
- moved on the sheet: S1, U1

Commit message: [PCB] Sent off for manufacturing
Parts:
- removed H1, H2, H3, H4: MOUNT-HOLE3.0, holes:MOUNT-HOLE3.0
Connections:
- new net SW2: R1.1, S2.2, U1.GP15
- new net SW3: R2.1, S3.2, U1.GP14
- net LEDDATA: now also U1.GP28; no longer U1.GP0
- net SCL: now also U1.GP21; no longer U1.GP17
- net SDA: now also U1.GP20; no longer U1.GP16
- net SW4: no longer R1.1, R2.1, S2.2, S3.2, U1.GP14, U1.GP15
Changed lines of the file:
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@@
 <part name="GND4" library="supply1" library_urn="urn:adsk.eagle:library:371" deviceset="GND" device=""/>
 <part name="GND5" library="supply1" library_urn="urn:adsk.eagle:library:371" deviceset="GND" device=""/>
-<part name="H1" library="holes" library_urn="urn:adsk.eagle:library:237" deviceset="MOUNT-HOLE" device="3.0" package3d_urn="urn:adsk.eagle:package:14277/1"/>
-<part name="H2" library="holes" library_urn="urn:adsk.eagle:library:237" deviceset="MOUNT-HOLE" device="3.0" package3d_urn="urn:adsk.eagle:package:14277/1"/>
-<part name="H3" library="holes" library_urn="urn:adsk.eagle:library:237" deviceset="MOUNT-HOLE" device="3.0" package3d_urn="urn:adsk.eagle:package:14277/1"/>
-<part name="H4" library="holes" library_urn="urn:adsk.eagle:library:237" deviceset="MOUNT-HOLE" device="3.0" package3d_urn="urn:adsk.eagle:package:14277/1"/>
 <part name="P+4" library="supply1" library_urn="urn:adsk.eagle:library:371" deviceset="VCC" device=""/>
 <part name="L5V" library="solpad" library_urn="urn:adsk.eagle:library:364" deviceset="LSP10" device="" package3d_urn="urn:adsk.eagle:package:26501/1"/>
@@
 <attribute name="VALUE" x="91.44" y="38.1" size="1.778" layer="96"/>
 </instance>
-<instance part="H1" gate="G$1" x="208.28" y="73.66" smashed="yes">
-<attribute name="NAME" x="210.312" y="74.2442" size="1.778" layer="95"/>
-<attribute name="VALUE" x="210.312" y="71.1962" size="1.778" layer="96"/>
-</instance>
-<instance part="H2" gate="G$1" x="243.84" y="73.66" smashed="yes">
-<attribute name="NAME" x="245.872" y="74.2442" size="1.778" layer="95"/>
-<attribute name="VALUE" x="245.872" y="71.1962" size="1.778" layer="96"/>
-</instance>
-<instance part="H3" gate="G$1" x="208.28" y="58.42" smashed="yes">
-<attribute name="NAME" x="210.312" y="59.0042" size="1.778" layer="95"/>
-<attribute name="VALUE" x="210.312" y="55.9562" size="1.778" layer="96"/>
-</instance>
-<instance part="H4" gate="G$1" x="243.84" y="58.42" smashed="yes">
-<attribute name="NAME" x="245.872" y="59.0042" size="1.778" layer="95"/>
-<attribute name="VALUE" x="245.872" y="55.9562" size="1.778" layer="96"/>
-</instance>
 <instance part="P+4" gate="VCC" x="55.88" y="88.9" smashed="yes">
 <attribute name="VALUE" x="53.34" y="86.36" size="1.778" layer="96" rot="R90"/>
@@
 </segment>
 <segment>
-<pinref part="U1" gate="U$1" pin="GP16"/>
-<wire x1="48.26" y1="30.48" x2="55.88" y2="30.48" width="0.1524" layer="91"/>
-<label x="53.34" y="30.48" size="1.778" layer="95"/>
+<wire x1="48.26" y1="43.18" x2="55.88" y2="43.18" width="0.1524" layer="91"/>
+<pinref part="U1" gate="U$1" pin="GP20"/>
+<label x="53.34" y="43.18" size="1.778" layer="95"/>
 </segment>
 </net>
@@
 </segment>
 <segment>
-<pinref part="U1" gate="U$1" pin="GP17"/>
-<wire x1="48.26" y1="33.02" x2="55.88" y2="33.02" width="0.1524" layer="91"/>
-<label x="53.34" y="33.02" size="1.778" layer="95"/>
+<wire x1="48.26" y1="45.72" x2="55.88" y2="45.72" width="0.1524" layer="91"/>
+<pinref part="U1" gate="U$1" pin="GP21"/>
+<label x="53.34" y="45.72" size="1.778" layer="95"/>
 </segment>
 </net>
@@
 <label x="5.08" y="38.1" size="1.778" layer="95"/>
 </segment>
+</net>
+<net name="LEDDATA" class="0">
+<segment>
+<pinref part="LD" gate="1" pin="MP"/>
+<wire x1="99.06" y1="20.32" x2="93.98" y2="20.32" width="0.1524" layer="91"/>
+<label x="88.9" y="20.32" size="1.778" layer="95"/>
+</segment>
+<segment>
+<pinref part="U1" gate="U$1" pin="GP28"/>
+<wire x1="48.26" y1="63.5" x2="55.88" y2="63.5" width="0.1524" layer="91"/>
+<label x="53.34" y="63.5" size="1.778" layer="95"/>
+</segment>
+</net>
+<net name="3V3" class="0">
+<segment>
+<pinref part="U1" gate="U$1" pin="3V3(OUT)"/>
+<wire x1="48.26" y1="83.82" x2="55.88" y2="83.82" width="0.1524" layer="91"/>
+<label x="53.34" y="83.82" size="1.778" layer="95"/>
+</segment>
+<segment>
+<pinref part="S2" gate="G$1" pin="1"/>
+<wire x1="154.94" y1="81.28" x2="149.86" y2="81.28" width="0.1524" layer="91"/>
+<label x="149.86" y="81.28" size="1.778" layer="95"/>
+</segment>
+<segment>
+<pinref part="S3" gate="G$1" pin="1"/>
+<wire x1="154.94" y1="53.34" x2="149.86" y2="53.34" width="0.1524" layer="91"/>
+<label x="149.86" y="53.34" size="1.778" layer="95"/>
+</segment>
+<segment>
+<pinref part="S4" gate="G$1" pin="1"/>
+<wire x1="154.94" y1="25.4" x2="149.86" y2="25.4" width="0.1524" layer="91"/>
+<label x="149.86" y="25.4" size="1.778" layer="95"/>
+</segment>
+<segment>
+<pinref part="A2" gate="A" pin="1"/>
+<wire x1="104.14" y1="53.34" x2="93.98" y2="53.34" width="0.1524" layer="91"/>
+<label x="93.98" y="53.34" size="1.778" layer="95"/>
+</segment>
+<segment>
+<pinref part="R4" gate="G$1" pin="1"/>
+<pinref part="R5" gate="G$1" pin="1"/>
+<wire x1="73.66" y1="50.8" x2="73.66" y2="48.26" width="0.1524" layer="91"/>
+<wire x1="73.66" y1="48.26" x2="68.58" y2="48.26" width="0.1524" layer="91"/>
+<junction x="73.66" y="48.26"/>
+<label x="68.58" y="48.26" size="1.778" layer="95"/>
+</segment>
+<segment>
+<pinref part="S1" gate="1" pin="O"/>
+<wire x1="132.08" y1="68.58" x2="134.62" y2="68.58" width="0.1524" layer="91"/>
+<label x="134.62" y="68.58" size="1.778" layer="95"/>
+</segment>
+</net>
+<net name="SW1" class="0">
+<segment>
+<pinref part="S1" gate="1" pin="P"/>
+<wire x1="124.46" y1="66.04" x2="119.38" y2="66.04" width="0.1524" layer="91"/>
+<label x="119.38" y="66.04" size="1.778" layer="95"/>
+</segment>
+<segment>
+<pinref part="U1" gate="U$1" pin="GP26"/>
+<wire x1="48.26" y1="55.88" x2="55.88" y2="55.88" width="0.1524" layer="91"/>
+<label x="53.34" y="55.88" size="1.778" layer="95"/>
+</segment>
+</net>
+<net name="SW3" class="0">
+<segment>
+<pinref part="U1" gate="U$1" pin="GP14"/>
+<wire x1="12.7" y1="33.02" x2="5.08" y2="33.02" width="0.1524" layer="91"/>
+<label x="5.08" y="33.02" size="1.778" layer="95"/>
+</segment>
 <segment>
 <wire x1="165.1" y1="53.34" x2="172.72" y2="53.34" width="0.1524" layer="91"/>
@@
 <label x="172.72" y="53.34" size="1.778" layer="95"/>
 </segment>
-<segment>
-<pinref part="U1" gate="U$1" pin="GP14"/>
-<wire x1="12.7" y1="33.02" x2="5.08" y2="33.02" width="0.1524" layer="91"/>
-<label x="5.08" y="33.02" size="1.778" layer="95"/>
+</net>
+<net name="SW2" class="0">
+<segment>
+<pinref part="U1" gate="U$1" pin="GP15"/>
+<wire x1="12.7" y1="30.48" x2="5.08" y2="30.48" width="0.1524" layer="91"/>
+<label x="5.08" y="30.48" size="1.778" layer="95"/>
 </segment>
 <segment>
@@
 <label x="172.72" y="81.28" size="1.778" layer="95"/>
 </segment>
-<segment>
-<pinref part="U1" gate="U$1" pin="GP15"/>
-<wire x1="12.7" y1="30.48" x2="5.08" y2="30.48" width="0.1524" layer="91"/>
-<label x="5.08" y="30.48" size="1.778" layer="95"/>
-</segment>
-</net>
-<net name="LEDDATA" class="0">
-<segment>
-<pinref part="U1" gate="U$1" pin="GP0"/>
-<wire x1="12.7" y1="78.74" x2="5.08" y2="78.74" width="0.1524" layer="91"/>
-<label x="5.08" y="78.74" size="1.778" layer="95"/>
-</segment>
-<segment>
-<pinref part="LD" gate="1" pin="MP"/>
-<wire x1="99.06" y1="20.32" x2="93.98" y2="20.32" width="0.1524" layer="91"/>
-<label x="88.9" y="20.32" size="1.778" layer="95"/>
-</segment>
-</net>
-<net name="3V3" class="0">
-<segment>
-<pinref part="U1" gate="U$1" pin="3V3(OUT)"/>
-<wire x1="48.26" y1="83.82" x2="55.88" y2="83.82" width="0.1524" layer="91"/>
-<label x="53.34" y="83.82" size="1.778" layer="95"/>
-</segment>
-<segment>
-<pinref part="S2" gate="G$1" pin="1"/>
-<wire x1="154.94" y1="81.28" x2="149.86" y2="81.28" width="0.1524" layer="91"/>
-<label x="149.86" y="81.28" size="1.778" layer="95"/>
-</segment>
-<segment>
-<pinref part="S3" gate="G$1" pin="1"/>
-<wire x1="154.94" y1="53.34" x2="149.86" y2="53.34" width="0.1524" layer="91"/>
-<label x="149.86" y="53.34" size="1.778" layer="95"/>
-</segment>
-<segment>
-<pinref part="S4" gate="G$1" pin="1"/>
-<wire x1="154.94" y1="25.4" x2="149.86" y2="25.4" width="0.1524" layer="91"/>
-<label x="149.86" y="25.4" size="1.778" layer="95"/>
-</segment>
-<segment>
-<pinref part="A2" gate="A" pin="1"/>
-<wire x1="104.14" y1="53.34" x2="93.98" y2="53.34" width="0.1524" layer="91"/>
-<label x="93.98" y="53.34" size="1.778" layer="95"/>
-</segment>
-<segment>
-<pinref part="R4" gate="G$1" pin="1"/>
-<pinref part="R5" gate="G$1" pin="1"/>
-<wire x1="73.66" y1="50.8" x2="73.66" y2="48.26" width="0.1524" layer="91"/>
-<wire x1="73.66" y1="48.26" x2="68.58" y2="48.26" width="0.1524" layer="91"/>
-<junction x="73.66" y="48.26"/>
-<label x="68.58" y="48.26" size="1.778" layer="95"/>
-</segment>
-<segment>
-<pinref part="S1" gate="1" pin="O"/>
-<wire x1="132.08" y1="68.58" x2="134.62" y2="68.58" width="0.1524" layer="91"/>
-<label x="134.62" y="68.58" size="1.778" layer="95"/>
-</segment>
-</net>
-<net name="SW1" class="0">
-<segment>
-<pinref part="S1" gate="1" pin="P"/>
-<wire x1="124.46" y1="66.04" x2="119.38" y2="66.04" width="0.1524" layer="91"/>
-<label x="119.38" y="66.04" size="1.778" layer="95"/>
-</segment>
-<segment>
-<pinref part="U1" gate="U$1" pin="GP26"/>
-<wire x1="48.26" y1="55.88" x2="55.88" y2="55.88" width="0.1524" layer="91"/>
-<label x="53.34" y="55.88" size="1.778" layer="95"/>
-</segment>
-</net>
+</net>
